File: pcb/pcb.kicad_pcb (KiCad board)
At the start: 2 copper layers, 40 x 30 mm, 10 parts, among them J1 PINHD_1x4_Male, J2 Conn_02x06_Odd_Even, SW1 SW_Push, SW2 SW_Push, SW3 SW_Push, U1 XIAO-ESP32

Commit message: Add AQStation & SensorBoard addons
Other:
- board text added: "XIAO Base for ESPHome"
- board text removed: "ESPHome XIAO Base"
Changed lines of the file:
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@@
 	(paper "A4")
 	(title_block
-		(title "ESPHome XIAO Base")
+		(title "XIAO Base for ESPHome")
 		(date "2025-03-26")
 		(rev "v1.00")
@@
 		)
 	)
-	(gr_text "ESPHome XIAO Base"
+	(gr_text "XIAO Base for ESPHome"
 		(at 50.48 34.47 90)
 		(layer "B.SilkS")
