File: pcb/pcb.kicad_sch (KiCad schematic)
At the start: 6 parts, among them J1 PINHD_1x4_Male, J2 Conn_02x06_Odd_Even, SW1 SW_Push, SW2 SW_Push, SW3 SW_Push, U1 XIAO-ESP32

Commit message: Update Schematics and PCB properties
Other:
- company: LambdaKB.dev -> 0rax
- title: LK5DK -> ESPHome XIAO Base
Changed lines of the file:
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@@
 	(paper "A4")
 	(title_block
-		(title "LK5DK")
-		(date "2025-03-23")
+		(title "ESPHome XIAO Base")
+		(date "2025-03-26")
 		(rev "v1.00")
-		(company "LambdaKB.dev")
-		(comment 1 "https://lambdakb.dev/devices/lk5dk")
+		(company "0rax")
+		(comment 1 "https://github.com/0rax/esphome-xiao-base/")
 	)
 	(rectangle

Commit message: Add AQStation & SensorBoard addons
Other:
- title: ESPHome XIAO Base -> XIAO Base for ESPHome
Changed lines of the file:
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@@
 	(paper "A4")
 	(title_block
-		(title "ESPHome XIAO Base")
+		(title "XIAO Base for ESPHome")
 		(date "2025-03-26")
 		(rev "v1.00")
