File: addons/aqstation/aqstation.kicad_sch (KiCad schematic)
At the start: 8 parts, among them J1 PMSA003, J2 Conn_02x06_Odd_Even, J3 Adafruit_I2C_Header, J5 RGB_Header, J6 Pimoroni_I2CGarden_Header, J7 StemmaQT_Qwiic_Header, J8 BME680_Header

Commit message: More compact version of the AQStation
Other:
- note added: "BME680_Header compatible with: - DFRobot Fermion BME680: https://www.dfrobot.com/product-2143.html - Adafruit BME680: https://www.adafruit.com/product/3660 - DFRobot Fermion BME688: https://www.dfrobot.com/product-2918.html - Adafruit BME688: https://www.adafruit.com/product/5046 Adafruit_I2C_Header compatible with: - Adafruit Si7021: https://www.adafruit.com/product/3251 - Adafruit MCP9808: http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"
- note removed: "Adafruit Style I2C Header w/ 2 Extra Pins Compatible with: - Adafruit Si7021: https://www.adafruit.com/product/3251 - Adafruit MCP9808: https://www.adafruit.com/product/1782 - Adafruit AHT20: https://www.adafruit.com/product/4566 - DFRobot Fermion SHT40: https://www.dfrobot.com/product-2437.html - DFRobot Fermion SHT31: https://www.dfrobot.com/product-2013.html - DFRobot Fermion SHTC3: https://ww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"
- note removed: "Compatible with Pimoroni I2C Breakout Garden: - Pimoroni BME680 Breakout: https://shop.pimoroni.com/products/bme680-breakout - Piomoroni MICS6814 Breakout: https://shop.pimoroni.com/products/mics6814-gas-sensor-breakout"
- note removed: "Compatible with: - DFRobot Fermion BME680: https://www.dfrobot.com/product-2143.html - Adabruit BME680: https://www.adafruit.com/product/3660 - DFRobot Fermion BME688: https://www.dfrobot.com/product-2918.html - Adafruit BME688: https://www.adafruit.com/product/5046"
Changed lines of the file:
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@@
-		)
-	)
-	(text "Adafruit Style I2C Header w/ 2 Extra Pins\n\nCompatible with:\n- Adafruit Si7021: https://www.adafruit.com/product/3251\n- Adafruit MCP9808: https://www.adafruit.com/product/1782\n- Adafruit AHT20: https://www.adafruit.com/product/4566\n- DFRobot Fermion SHT40: https://www.dfrobot.com/product-2437.html\n- DFRobot Fermion SHT31: https://www.dfrobot.com/product-2013.html\n- DFRobot Fermion SHTC3: https://www.dfrobot.com/product-2436.html\n- DFRobot Fermion AHT20: https://www.dfrobot.com/product-2603.html\n- DFRobot Fermion SHT35: https://www.dfrobot.com/product-2016.html\n\nMaybe:\n- CJMCU-8128 CCS811+SI7021+BMP280: https://aliexpress.com/item/1005008633429391.html\n- ENS160+AHT21 Module: https://aliexpress.com/item/1005004761725413.html\n- BME680 Purple Breakout: https://www.studiopieters.nl/bme680-gas-sensor/\n    (pinout needs to be verified, but the left 4 holes should match I2C header)"
-		(exclude_from_sim no)
-		(at 110.744 71.12 0)
-		(effects
-			(font
-				(size 1.27 1.27)
-			)
-			(justify left top)
 		)
 	)
@@
 		)
 	)
-	(text "Compatible with:\n- DFRobot Fermion BME680: https://www.dfrobot.com/product-2143.html\n- Adabruit BME680: https://www.adafruit.com/product/3660\n- DFRobot Fermion BME688: https://www.dfrobot.com/product-2918.html\n- Adafruit BME688: https://www.adafruit.com/product/5046"
+	(text "BME680_Header compatible with:\n- DFRobot Fermion BME680: https://www.dfrobot.com/product-2143.html\n- Adafruit BME680: https://www.adafruit.com/product/3660\n- DFRobot Fermion BME688: https://www.dfrobot.com/product-2918.html\n- Adafruit BME688: https://www.adafruit.com/product/5046\n\nAdafruit_I2C_Header compatible with:\n- Adafruit Si7021: https://www.adafruit.com/product/3251\n- Adafruit MCP9808: https://www.adafruit.com/product/1782\n- Adafruit AHT20: https://www.adafruit.com/product/4566\n- DFRobot Fermion SHT40: https://www.dfrobot.com/product-2437.html\n- DFRobot Fermion SHT31: https://www.dfrobot.com/product-2013.html\n- DFRobot Fermion SHTC3: https://www.dfrobot.com/product-2436.html\n- DFRobot Fermion AHT20: https://www.dfrobot.com/product-2603.html\n- DFRobot Fermion SHT35: https://www.dfrobot.com/product-2016.html\n- BME680 Purple Breakout: https://www.studiopieters.nl/bme680-gas-sensor/\n\nPimoroni_I2CGarden_Header compatible with:\n- Pimoroni BME680 Breakout: https://shop.pimoroni.com/products/bme680-breakout\n- Pimoroni MICS6814 Breakout: https://shop.pimoroni.com/products/mics6814-gas-sensor-breakout"
 		(exclude_from_sim no)
 		(at 110.49 52.578 0)
 		(effects
 			(font
-				(size 1.27 1.27)
-			)
-			(justify left top)
-		)
-	)
-	(text "Compatible with Pimoroni I2C Breakout Garden:\n- Pimoroni BME680 Breakout: https://shop.pimoroni.com/products/bme680-breakout\n- Piomoroni MICS6814 Breakout: https://shop.pimoroni.com/products/mics6814-gas-sensor-breakout"
-		(exclude_from_sim no)
-		(at -63.5 70.612 0)
-		(effects
-			(font

Commit message: Finalize aqstation
Parts:
- renumbered J2 to J1, J1 to J2, J6 to J4, J8 to J5, J7 to J6, J5 to J7
Other:
- note added: "RGB LED Header"
- note added: "ST/Qwiic Connectors"
- note added: "Sensor"
- note removed: "Compatible with any 5V WS2812B Compatible LED strips."
- moved on the sheet: J1, J2, J3, J4, J5, J6, J7, R2

Commit message: Fix issues with the initial version and add support for DFRobot BME breakouts
Update documentation
Parts:
- removed J4: Pimoroni_I2CGarden_Header, Header:Pimoroni_I2CGarden_Header, symbol Header:Pimoroni_I2CGarden_Header
- added J4: Adafruit_I2C_Header, Header:Adafruit_I2C_Header, symbol Header:Adafruit_I2C_Header
- J3: value Adafruit_I2C_Header -> DFRobot_BME680_Header; footprint Header:Adafruit_I2C_Header -> Header:DFRobot_BME680_Header; symbol Header:Adafruit_I2C_Header -> Header:DFRobot_BME680_Header
- J5: value BME680_Header -> Adafruit_BME680_Header; footprint Header:BME680_Header -> Header:Adafruit_BME680_Header; symbol Header:BME680_Header -> Header:Adafruit_BME680_Header
Connections:
- net D9 is gone; now on net ADDR: J1.8 (D8), J3.6 (MI)
- net +3.3V: now also J3.1 (VCC), J4.2 (VCC); no longer J3.2 (VCC)
- net GND: now also J3.2 (GND), J4.3 (GND); no longer J3.3 (GND)
- net SCL: now also J3.5 (SCK), J4.4 (SCL); no longer J3.4 (SCL)
- net SDA: now also J3.3 (MO), J4.5 (SDA); no longer J3.5 (SDA)
- net ADDR: now reaches J5.5 (SDO)
- net ADDR: now also J4.6 (IO1)
- net EN: now reaches J5.7 (CS)
- net EN: now also J1.6 (D3), J3.4 (CS), J4.7 (IO2)
- removed net D10: J1.6 (D10), J3.7 (IO2)
- net D3 renamed SET
- net D8 renamed LEDIO
- no-connect marks 6 -> 4
Other:
- note added: "Adafruit_I2C_Header compatible with: - Adafruit Si7021: https://www.adafruit.com/product/3251 - Adafruit MCP9808: https://www.adafruit.com/product/1782 - Adafruit AHT20: https://www.adafruit.com/product/4566 - DFRobot Fermion SHT40: https://www.dfrobot.com/product-2437.html - DFRobot Fermion SHT31: https://www.dfrobot.com/product-2013.html - DFRobot Fermion SHTC3: https://www.dfrobot.com/product-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"
- note removed: "BME680_Header compatible with: - DFRobot Fermion BME680: https://www.dfrobot.com/product-2143.html - Adafruit BME680: https://www.adafruit.com/product/3660 - DFRobot Fermion BME688: https://www.dfrobot.com/product-2918.html - Adafruit BME688: https://www.adafruit.com/product/5046 Adafruit_I2C_Header compatible with: - Adafruit Si7021: https://www.adafruit.com/product/3251 - Adafruit MCP9808: http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"
