File: addons/sensorboard/sensorboard.kicad_pcb (KiCad board)
At the start: 2 copper layers, 60 x 60 mm, 21 parts, among them J1 Conn_02x06_Odd_Even, J10 Adafruit_I2C_Header, J11 BME680_Header, J12 RGB_Header, J2 SparkFun_I2C_Header, J3 Adafruit_I2C_Header, J4 Pimoroni_I2CGarden_Header, J5 Pimoroni_I2CGarden_Header, J6 Adafruit_I2C_Header, J7 SparkFun_I2C_Header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

Commit message: Finalize aqstation
Other:
- board text added: "0.1600 mm / 0.1600 mm"
- board text added: "0.3000 mm"
- board text added: "1.6000 mm"
- board text added: "2"
- board text added: "60.0000 mm x 60.0000 mm"
- board text added: "BOARD CHARACTERISTICS"
- board text added: "Board Thickness:"
- board text added: "Board overall dimensions:"
- board text added: "Castellated pads:"
- board text added: "Copper Finish:"
- board text added: "Copper Layer Count:"
- board text added: "Edge card connectors:"
- board text added: "HAL lead-free"
- board text added: "Impedance Control:"
- board text added: "Min hole diameter:"
- board text added: "Min track/spacing:"
- board text added: "No"
- board text added: "Plated Board Edge:"

Commit message: Fix issues with the initial version and add support for DFRobot BME breakouts
Update documentation
Parts:
- J11: value BME680_Header -> Adafruit_BME680_Header; footprint Header:BME680_Header -> Header:Adafruit_BME680_Header
Connections:
- J11 pad 5: unconnected-(J11-SDO-Pad5) -> /D6
- J11 pad 7: unconnected-(J11-CS-Pad7) -> /D7
Routing:
- net /D7: track 40.7 -> 61.7 mm
- net /D6: track 38.0 -> 57.3 mm
- net GND: track 51.0 -> 55.2 mm
- net +3.3V: track 201.9 -> 203.1 mm
Other:
- board text added: "Adafruit BME280 & BME680X (StemmaQT)"
- board text added: "Sensor 3 Compatibility"
- board text removed: "Adafruit BME28X/68X DFRobot Fermion BME680"
